File: kicad/factotum/inputs.sch (KiCad schematic (older format))
At the start: 29 parts

Commit message: working on schematic
Parts:
- removed D? (x3): D_TVS, symbol Device:D_TVS
- added C21, C24, C28: 33n, symbol Device:C_Small
- added C25, C27: 100n, symbol Device:C_Small
- added J4: Conn_01x10_Female, symbol Connector:Conn_01x10_Female
- added J6: Conn_01x10_Male, symbol Connector:Conn_01x10_Male
- added R16, R20, R24: 100, symbol Device:R_Small
- C20, C22, C23, C26: renamed from C?; value 100n -> 33n
- U5: renamed from U?; value MCP6004 -> ADC128S022
- gave numbers to parts that had none: 14
- renumbered FRQ to FRQ1, OFF to OFF1, SCL to SCL1, SEL to SEL1
Connections:
- net +3.3VA: now also C25.1, J4.1 (Pin_1), J6.1 (Pin_1)
- net +3V3: now also C27.1
- net ADC_CLK: now also U5.10 (IN6), C28.1, R24.1; no longer R23.1, U4.8, U5.9 (IN5)
- net ADC_VOCT: now also C21.1, R16.1; no longer R15.1, U4.1
- net GND: now also C21.2, C24.2, C25.2, C27.2, C28.2, J4.10 (Pin_10), J6.10 (Pin_10)
- net B_SCALE: now reaches R18.2
- net B_SCALE: now also J6.7 (Pin_7); no longer J7.S
- net B_CLK: now reaches R22.2
- net B_CLK: now also J6.8 (Pin_8); no longer J8.S
- net B_VOCT: now reaches R14.2
- net B_VOCT: now also J6.6 (Pin_6); no longer J5.S
- net ADC_FRQ renamed T_FRQ
- net T_FRQ: now also J4.2 (Pin_2); no longer U5.4 (IN0)
- net ADC_OFF renamed T_OFF
- net T_OFF: now also J4.5 (Pin_5); no longer U5.10 (IN6), U5.7 (IN3)
- removed net ADC_SCL: C23.1, R19.1, SCL1.2, U4.7, U5.6 (IN2)
- net ADC_SEL renamed T_SEL
- net T_SEL: now also J4.3 (Pin_3); no longer U5.5 (IN1)
- net SW_MODE renamed T_MODE
- net T_MODE: now also J4.9 (Pin_9)
- new net: R15.1, R16.2, U4.1
- new net: R19.1, R20.2, U4.7
- new net: R23.1, R24.2, U4.8
- new net ADC_VC_SCL: C24.1, R20.1, U5.9 (IN5)
- new net B_FRQ: J6.2 (Pin_2), U5.4 (IN0)
- new net B_MODE: J6.9 (Pin_9)
- new net B_OFF: J6.5 (Pin_5), U5.7 (IN3)
- new net B_SCL: J6.4 (Pin_4), U5.6 (IN2)
- new net B_SEL: J6.3 (Pin_3), U5.5 (IN1)
- new net T_CLK: J4.8 (Pin_8), J8.S
- new net T_SCALE: J4.7 (Pin_7), J7.S
- new net T_SCL: C23.1, J4.4 (Pin_4), SCL1.2
- new net T_VOCT: J4.6 (Pin_6), J5.S
Other:
- moved on the sheet: C20, C22, C23, C26, J5, J7, J8, R13, R14, R15, R17, R18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
