File: kicad/factotum/factotum.sch (KiCad schematic (older format))
At the start: 27 parts, among them J1 Conn_01x06, J2 USART, U1 STM32F411RETx, U8 M24C02-RMN, Y1 16 MHz

Commit message: more work on routing
Parts:
- added J? (x2): Conn_01x08_Female, Connector_PinSocket_2.54mm:PinSocket_1x08_P2.54mm_Vertical, symbol Connector:Conn_01x08_Female
- added J? (x2): Conn_01x08_Male, Connector_PinHeader_2.54mm:PinHeader_1x08_P2.54mm_Vertical, symbol Connector:Conn_01x08_Male
- added J?: Conn_01x05_Female, Connector_PinSocket_2.54mm:PinSocket_1x05_P2.54mm_Vertical, symbol Connector:Conn_01x05_Female
- added J?: Conn_01x05_Male, Connector_PinHeader_2.54mm:PinHeader_1x05_P2.54mm_Vertical, symbol Connector:Conn_01x05_Male
- added J?: Conn_01x17_Female, Connector_PinSocket_2.54mm:PinSocket_1x17_P2.54mm_Vertical, symbol Connector:Conn_01x17_Female
- added J?: Conn_01x17_Male, Connector_PinHeader_2.54mm:PinHeader_1x17_P2.54mm_Vertical, symbol Connector:Conn_01x17_Male
Connections:
- net +3.3VA: now also J?.3 (Pin_3), J?.3 (Pin_3)
- net +3V3: now also J?.9 (Pin_9), J?.9 (Pin_9)
- net B_CLK_SW: now also J?.4 (Pin_4)
- net B_MODE_SW: now also J?.7 (Pin_7)
- net B_RST_SW: now also J?.6 (Pin_6)
- net B_VOCT_SW: now also J?.2 (Pin_2)
- net GND: now also J?.8 (Pin_8), J?.8 (Pin_8)
- new net B_1: J?.1 (Pin_1)
- new net B_2: J?.2 (Pin_2)
- new net B_3: J?.3 (Pin_3)
- new net B_4: J?.4 (Pin_4)
- new net B_5: J?.5 (Pin_5)
- new net B_6: J?.6 (Pin_6)
- new net B_7: J?.7 (Pin_7)
- new net B_8: J?.8 (Pin_8)
- new net B_CLK: J?.3 (Pin_3)
- new net B_FRQ: J?.1 (Pin_1)
- new net B_OFF: J?.2 (Pin_2)
- new net B_RST: J?.5 (Pin_5)
- new net B_SCL: J?.4 (Pin_4)
- new net B_SEL: J?.5 (Pin_5)
- new net B_VOCT: J?.1 (Pin_1)
- new net G1_B: J?.3 (Pin_3)
- new net G1_T: J?.3 (Pin_3)
- new net G2_B: J?.1 (Pin_1)
- new net G2_T: J?.1 (Pin_1)
- new net G3_B: J?.16 (Pin_16)
- new net G3_T: J?.16 (Pin_16)
- new net G4_B: J?.14 (Pin_14)
- new net G4_T: J?.14 (Pin_14)
- new net G5_B: J?.12 (Pin_12)
- new net G5_T: J?.12 (Pin_12)
- new net G6_B: J?.10 (Pin_10)
- new net G6_T: J?.10 (Pin_10)
- new net G7_B: J?.7 (Pin_7)
- new net G7_T: J?.7 (Pin_7)
- new net G8_B: J?.5 (Pin_5)
- new net G8_T: J?.5 (Pin_5)
- new net R1_B: J?.4 (Pin_4)
- new net R1_T: J?.4 (Pin_4)
- new net R2_B: J?.2 (Pin_2)
- new net R2_T: J?.2 (Pin_2)
- new net R3_B: J?.17 (Pin_17)
- new net R3_T: J?.17 (Pin_17)
- new net R4_B: J?.15 (Pin_15)
- new net R4_T: J?.15 (Pin_15)
- new net R5_B: J?.13 (Pin_13)
- new net R5_T: J?.13 (Pin_13)
- new net R6_B: J?.11 (Pin_11)
- new net R6_T: J?.11 (Pin_11)
- new net R7_B: J?.8 (Pin_8)
- new net R7_T: J?.8 (Pin_8)
- new net R8_B: J?.6 (Pin_6)
- new net R8_T: J?.6 (Pin_6)
- new net T_1: J?.1 (Pin_1)
- new net T_2: J?.2 (Pin_2)
- new net T_3: J?.3 (Pin_3)
- new net T_4: J?.4 (Pin_4)
- new net T_5: J?.5 (Pin_5)
- new net T_6: J?.6 (Pin_6)
- new net T_7: J?.7 (Pin_7)
- new net T_8: J?.8 (Pin_8)
- new net T_CLK: J?.3 (Pin_3)
- new net T_CLK_SW: J?.4 (Pin_4)
- new net T_FRQ: J?.1 (Pin_1)
- new net T_MODE_SW: J?.7 (Pin_7)
- new net T_OFF: J?.2 (Pin_2)
- new net T_RST: J?.5 (Pin_5)
- new net T_RST_SW: J?.6 (Pin_6)
- new net T_SCL: J?.4 (Pin_4)
- new net T_SEL: J?.5 (Pin_5)
- new net T_VOCT: J?.1 (Pin_1)
- new net T_VOCT_SW: J?.2 (Pin_2)

Commit message: finished routing
Parts:
- gave numbers to parts that had none: 8
Connections:
- net B_MODE_SW: now also U1.50 (PA15); no longer U1.14 (PA0)
Changed lines of the file:
@@
 NoConn ~ 6300 3050
 NoConn ~ 6300 3150
-NoConn ~ 6300 3450
 NoConn ~ 6300 3750
 NoConn ~ 6300 3850
@@
 Wire Wire Line
 	4800 3650 4900 3650
-Text GLabel 6300 1950 2    50   Input ~ 0
+Text GLabel 6300 3450 2    50   Input ~ 0
 B_MODE_SW
 $Comp
@@
 P 1300 5100
 AR Path="/6088BCB1/60187068" Ref="J?"  Part="1"
-AR Path="/60187068" Ref="J?"  Part="1"
-F 0 "J?" H 1150 5550 50  0000 L CNN
+AR Path="/60187068" Ref="J4"  Part="1"
+F 0 "J4" H 1150 5550 50  0000 L CNN
 F 1 "Conn_01x08_Female" V 1350 4700 50  0000 L CNN
 F 2 "Connector_PinSocket_2.54mm:PinSocket_1x08_P2.54mm_Vertical" H 1300 5100 50  0001 C CNN
@@
 P 1650 5100
 AR Path="/6088BCB1/6018706E" Ref="J?"  Part="1"
-AR Path="/6018706E" Ref="J?"  Part="1"
-F 0 "J?" H 1800 5550 50  0000 C CNN
+AR Path="/6018706E" Ref="J18"  Part="1"
+F 0 "J18" H 1800 5550 50  0000 C CNN
 F 1 "Conn_01x08_Male" V 1600 5050 50  0000 C CNN
 F 2 "Connector_PinHeader_2.54mm:PinHeader_1x08_P2.54mm_Vertical" H 1650 5100 50  0001 C CNN
@@
 P 850 6200
 AR Path="/606FF2F2/6019FE4A" Ref="#PWR?"  Part="1"
-AR Path="/6019FE4A" Ref="#PWR?"  Part="1"
-F 0 "#PWR?" H 850 6050 50  0001 C CNN
+AR Path="/6019FE4A" Ref="#PWR0101"  Part="1"
+F 0 "#PWR0101" H 850 6050 50  0001 C CNN
 F 1 "+3.3VA" H 865 6373 50  0000 C CNN
 F 2 "" H 850 6200 50  0001 C CNN
@@
 P 2250 6200
 AR Path="/606FF2F2/6019FE50" Ref="#PWR?"  Part="1"
-AR Path="/6019FE50" Ref="#PWR?"  Part="1"
-F 0 "#PWR?" H 2250 6050 50  0001 C CNN
+AR Path="/6019FE50" Ref="#PWR0102"  Part="1"
+F 0 "#PWR0102" H 2250 6050 50  0001 C CNN
 F 1 "+3.3VA" H 2265 6373 50  0000 C CNN
 F 2 "" H 2250 6200 50  0001 C CNN
@@
 $EndComp
 $Comp
-L power:GND #PWR?
+L power:GND #PWR0103
 U 1 1 6019FE56
 P 850 7600
-AR Path="/6019FE56" Ref="#PWR?"  Part="1"
+AR Path="/6019FE56" Ref="#PWR0103"  Part="1"
 AR Path="/606FF2F2/6019FE56" Ref="#PWR?"  Part="1"
-F 0 "#PWR?" H 850 7350 50  0001 C CNN
+F 0 "#PWR0103" H 850 7350 50  0001 C CNN
 F 1 "GND" V 950 7650 50  0000 R CNN
 F 2 "" H 850 7600 50  0001 C CNN
@@
 $EndComp
 $Comp
-L power:GND #PWR?
+L power:GND #PWR0104
 U 1 1 6019FE5C
 P 2200 7600
-AR Path="/6019FE5C" Ref="#PWR?"  Part="1"
+AR Path="/6019FE5C" Ref="#PWR0104"  Part="1"
 AR Path="/606FF2F2/6019FE5C" Ref="#PWR?"  Part="1"
-F 0 "#PWR?" H 2200 7350 50  0001 C CNN
+F 0 "#PWR0104" H 2200 7350 50  0001 C CNN
 F 1 "GND" V 2100 7650 50  0000 R CNN
 F 2 "" H 2200 7600 50  0001 C CNN
@@
 P 1350 6200
 AR Path="/606FF2F2/6019FE64" Ref="J?"  Part="1"
-AR Path="/6019FE64" Ref="J?"  Part="1"
-F 0 "J?" H 1200 6500 50  0000 L CNN
+AR Path="/6019FE64" Ref="J6"  Part="1"
+F 0 "J6" H 1200 6500 50  0000 L CNN
 F 1 "Conn_01x05_Female" V 1400 6000 50  0000 L CNN
 F 2 "Connector_PinSocket_2.54mm:PinSocket_1x05_P2.54mm_Vertical" H 1350 6200 50  0001 C CNN
@@
 P 1700 6200
 AR Path="/606FF2F2/6019FE6A" Ref="J?"  Part="1"
-AR Path="/6019FE6A" Ref="J?"  Part="1"
-F 0 "J?" H 1750 6500 50  0000 C CNN
+AR Path="/6019FE6A" Ref="J19"  Part="1"
+F 0 "J19" H 1750 6500 50  0000 C CNN
 F 1 "Conn_01x05_Male" V 1600 6300 50  0000 C CNN
 F 2 "Connector_PinHeader_2.54mm:PinHeader_1x05_P2.54mm_Vertical" H 1700 6200 50  0001 C CNN
@@
 P 1350 7200
 AR Path="/606FF2F2/6019FE72" Ref="J?"  Part="1"
-AR Path="/6019FE72" Ref="J?"  Part="1"
-F 0 "J?" H 1250 7600 50  0000 L CNN
-F 1 "Conn_01x08_Female" V 1650 6800 50  0000 L CNN
+AR Path="/6019FE72" Ref="J13"  Part="1"
+F 0 "J13" H 1250 7600 50  0000 L CNN
+F 1 "Conn_01x08_Female" V 1400 6800 50  0000 L CNN
 F 2 "Connector_PinSocket_2.54mm:PinSocket_1x08_P2.54mm_Vertical" H 1350 7200 50  0001 C CNN
 F 3 "~" H 1350 7200 50  0001 C CNN
@@
 P 1700 7200
 AR Path="/606FF2F2/6019FE78" Ref="J?"  Part="1"
-AR Path="/6019FE78" Ref="J?"  Part="1"
-F 0 "J?" H 1800 7600 50  0000 C CNN
-F 1 "Conn_01x08_Male" V 1400 7200 50  0000 C CNN
+AR Path="/6019FE78" Ref="J20"  Part="1"
+F 0 "J20" H 1800 7600 50  0000 C CNN
+F 1 "Conn_01x08_Male" V 1650 7150 50  0000 C CNN
 F 2 "Connector_PinHeader_2.54mm:PinHeader_1x08_P2.54mm_Vertical" H 1700 7200 50  0001 C CNN
 F 3 "~" H 1700 7200 50  0001 C CNN
@@
 P 4550 6500
 AR Path="/6088BCB1/601C955B" Ref="#PWR?"  Part="1"
-AR Path="/601C955B" Ref="#PWR?"  Part="1"
-F 0 "#PWR?" H 4550 6350 50  0001 C CNN
+AR Path="/601C955B" Ref="#PWR0106"  Part="1"
+F 0 "#PWR0106" H 4550 6350 50  0001 C CNN
 F 1 "+3.3V" H 4565 6673 50  0000 C CNN
 F 2 "" H 4550 6500 50  0001 C CNN
@@
 P 3250 6500
 AR Path="/6088BCB1/601C9561" Ref="#PWR?"  Part="1"
-AR Path="/601C9561" Ref="#PWR?"  Part="1"
-F 0 "#PWR?" H 3250 6350 50  0001 C CNN
+AR Path="/601C9561" Ref="#PWR0107"  Part="1"
+F 0 "#PWR0107" H 3250 6350 50  0001 C CNN
 F 1 "+3.3V" H 3265 6673 50  0000 C CNN
 F 2 "" H 3250 6500 50  0001 C CNN
@@
 P 3700 6500
 AR Path="/6088BCB1/601C9567" Ref="J?"  Part="1"
-AR Path="/601C9567" Ref="J?"  Part="1"
-F 0 "J?" H 3592 5475 50  0000 C CNN
+AR Path="/601C9567" Ref="J21"  Part="1"
+F 0 "J21" H 3592 5475 50  0000 C CNN
 F 1 "Conn_01x17_Female" V 3750 6400 50  0000 C CNN
 F 2 "Connector_PinSocket_2.54mm:PinSocket_1x17_P2.54mm_Vertical" H 3700 6500 50  0001 C CNN
@@
 P 4050 6500
 AR Path="/6088BCB1/601C956D" Ref="J?"  Part="1"
-AR Path="/601C956D" Ref="J?"  Part="1"
-F 0 "J?" H 4150 5600 50  0000 R CNN
+AR Path="/601C956D" Ref="J22"  Part="1"
+F 0 "J22" H 4150 5600 50  0000 R CNN
 F 1 "Conn_01x17_Male" V 4000 6750 50  0000 R CNN
 F 2 "Connector_PinHeader_2.54mm:PinHeader_1x17_P2.54mm_Vertical" H 4050 6500 50  0001 C CNN
@@
 Wire Wire Line
 	3500 6500 3250 6500
+NoConn ~ 6300 1950
 $EndSCHEMATC
